File: hardware/vers0.9/gerador_sinais.kicad_sch (KiCad schematic)
At the start: 6 parts, among them J1 Conn_02x03_Odd_Even, J2 Conn_02x05_Odd_Even, J3 Conn_01x03, U2 74HC138

Commit message: 250330-0836
Parts:
- removed U2: 74HC138, symbol 74xx:74HC138
Connections:
- net AD_SYSCLK renamed DISPLAY_SCLK
- net D0 renamed DDS_DATA
- net D1 renamed DDS_W_CLK
- net D2 renamed DDS_FQ_UD
- net D3 renamed DISPLAY_CS
- net D4 renamed SHREG_HOLD
- net D5 renamed SHREG_DIN
- net D6 renamed SHREG_CLK
- net D7 renamed SHREG_DOUT
- net DEMUX_A renamed ADC
- net DEMUX_B renamed DDS_ADJ
- net DEMUX_C renamed DISPLAY_SID
- net DEMUX_G1: no longer names the net of U1.25 (GPIO19)
- net LATCH_OC renamed RESET
- net LED renamed PWM

Commit message: 250404-0705
Parts:
- added J7: Fonte 5v, symbol Connector_Generic:Conn_01x02
- added J8, J9: Fonte 12V, symbol Connector_Generic:Conn_01x02
- added R1: 10K, symbol Device:R
- added U4, U5, U8, U9: 74HC00, symbol 74xx:74HC00
- J1: value Conn_02x03_Odd_Even -> COMUNIC
- J2: value Conn_02x05_Odd_Even -> JTAG
Connections:
- net SHREG_DIN is gone; now on net ADC: U1.6 (GPIO27)
- net 3,3V: now also R1.1
- net ADC: no longer U1.7 (GPIO26)
- net GND: now also J7.2 (Pin_2), J8.2 (Pin_2), J9.1 (Pin_1), U4.1, U4.2, U8.1, U8.2, U9.1, U9.2
- net RESET: now also R1.2, U5.1, U5.2
- net SHREG_CLK: now also U1.25 (GPIO19); no longer U1.10 (GPIO32)
- net at J3.3 (Pin_3): now also J7.1 (Pin_1)
- net DDS_W_CLK renamed DDS_WCLK
- net DISPLAY_CS renamed SHREG_DATAIN
- net DISPLAY_SCLK renamed DISPLAY_CLK
- net DISPLAY_SID renamed DISPLAY_DATA
- net SHREG_DOUT renamed SHREG_DATAOUT
- new net -12V: J9.2 (Pin_2)
- new net 12V: J8.1 (Pin_1)
- new net /RESET: U5.3
Other:
- added sheet DDS (DDS.kicad_sch)
- note added: "+"
- note added: "-"
- moved on the sheet: C1, J1

Commit message: 250425-1655
Connections:
- net DDS_DATA: now also U1.9 (GPIO33); no longer U1.20 (GPIO4)
- net SHREG_DATAOUT: now also U1.20 (GPIO4); no longer U1.9 (GPIO33)

Commit message: 250427-1145
Connections:
- net at J1.5 (Pin_5): now also U1.15 (EN)
Other:
- moved on the sheet: C1
Changed lines of the file:
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@@
 	(wire
 		(pts
-			(xy 203.2 88.9) (xy 210.82 88.9)
+			(xy 203.2 88.9) (xy 234.95 88.9)
 		)
 		(stroke
@@
 	(wire
 		(pts
+			(xy 173.99 81.28) (xy 173.99 54.61)
+		)
+		(stroke
+			(width 0)
+			(type default)
+		)
+	)
+	(wire
+		(pts
 			(xy 107.95 19.05) (xy 107.95 24.13)
 		)
@@
 	(wire
 		(pts
+			(xy 109.22 71.12) (xy 113.03 71.12)
+		)
+		(stroke
+			(width 0)
+			(type default)
+		)
+	)
+	(wire
+		(pts
 			(xy 86.36 29.21) (xy 86.36 34.29)
 		)
@@
 	(wire
 		(pts
+			(xy 109.22 54.61) (xy 109.22 71.12)
+		)
+		(stroke
+			(width 0)
+			(type default)
+		)
+	)
+	(wire
+		(pts
 			(xy 53.34 34.29) (xy 38.1 34.29)
 		)
@@
 	(wire
 		(pts
+			(xy 173.99 54.61) (xy 109.22 54.61)
+		)
+		(stroke
+			(width 0)
+			(type default)
+		)
+	)
+	(wire
+		(pts
 			(xy 139.7 96.52) (xy 156.21 96.52)
 		)
@@
 	(wire
 		(pts
-			(xy 22.86 43.18) (xy 22.86 49.53)
+			(xy 240.03 140.97) (xy 240.03 147.32)
 		)
 		(stroke
@@
 	(wire
 		(pts
-			(xy 22.86 29.21) (xy 22.86 35.56)
+			(xy 240.03 127) (xy 240.03 133.35)
 		)
 		(stroke
@@
 		(pts
 			(xy 203.2 69.85) (xy 203.2 74.93)
+		)
+		(stroke
+			(width 0)
+			(type default)
+		)
+	)
+	(wire
+		(pts
+			(xy 176.53 81.28) (xy 173.99 81.28)
 		)
 		(stroke
@@
 	(global_label "RESET"
 		(shape output)
-		(at 210.82 88.9 0)
+		(at 234.95 88.9 0)
 		(fields_autoplaced yes)
 		(effects
@@
 		)
 		(property "Intersheetrefs" "${INTERSHEET_REFS}"
-			(at 219.5503 88.9 0)
+			(at 243.6803 88.9 0)
 			(effects
 				(font
@@
 	(symbol
 		(lib_id "Device:C")
-		(at 22.86 39.37 0)
+		(at 240.03 137.16 0)
 		(unit 1)
 		(exclude_from_sim no)
@@
 		(fields_autoplaced yes)
 		(property "Reference" "C1"
-			(at 26.67 38.0999 0)
+			(at 243.84 135.8899 0)
 			(effects
 				(font
@@
 		)
 		(property "Value" "100nF"
-			(at 26.67 40.6399 0)
+			(at 243.84 138.4299 0)
 			(effects
 				(font
@@
 		)
 		(property "Footprint" ""
-			(at 23.8252 43.18 0)
+			(at 240.9952 140.97 0)
 			(effects
 				(font
@@
 		)
 		(property "Datasheet" "~"
-			(at 22.86 39.37 0)
+			(at 240.03 137.16 0)
 			(effects
 				(font
@@
 		)
 		(property "Description" "Unpolarized capacitor"
-			(at 22.86 39.37 0)
+			(at 240.03 137.16 0)
 			(effects
 				(font
@@
 	(symbol
 		(lib_id "power:VCC")
-		(at 22.86 29.21 0)
+		(at 240.03 127 0)
 		(unit 1)
 		(exclude_from_sim no)
@@
 		(dnp no)
 		(property "Reference" "#PWR12"
-			(at 22.86 33.02 0)
+			(at 240.03 130.81 0)
 			(effects
 				(font
@@
 		)
 		(property "Value" "3,3V"
-			(at 22.86 24.13 0)
+			(at 240.03 121.92 0)
 			(effects
 				(font
@@
 		)
 		(property "Footprint" ""
-			(at 22.86 29.21 0)
+			(at 240.03 127 0)
 			(effects
 				(font
@@
 		)
 		(property "Datasheet" ""
-			(at 22.86 29.21 0)
+			(at 240.03 127 0)
 			(effects
 				(font
@@
 		)
 		(property "Description" "Power symbol creates a global label with name \"VCC\""
-			(at 22.86 29.21 0)
+			(at 240.03 127 0)
 			(effects
 				(font
@@
 	(symbol
 		(lib_id "power:GND")
-		(at 22.86 49.53 0)
+		(at 240.03 147.32 0)
 		(unit 1)
 		(exclude_from_sim no)
@@
 		(fields_autoplaced yes)
 		(property "Reference" "#PWR11"
-			(at 22.86 55.88 0)
+			(at 240.03 153.67 0)
 			(effects
 				(font
@@
 		)
 		(property "Value" "GND"
-			(at 22.86 54.61 0)
+			(at 240.03 152.4 0)
 			(effects
 				(font
@@
 		)
 		(property "Footprint" ""
-			(at 22.86 49.53 0)
+			(at 240.03 147.32 0)
 			(effects
 				(font
@@
 		)
 		(property "Datasheet" ""
-			(at 22.86 49.53 0)
+			(at 240.03 147.32 0)
 			(effects
 				(font
@@
 		)
 		(property "Description" "Power symbol creates a global label with name \"GND\" , ground"
-			(at 22.86 49.53 0)
-			(effects
-				(font
+			(at 240.03 147.32 0)
+			(effects
+				(font

Commit message: 250826-1410
Connections:
- net DISPLAY_CS: now reaches U1.10 (GPIO32)
Changed lines of the file:
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@@
+	(wire
+		(pts
+			(xy 91.44 83.82) (xy 113.03 83.82)
+		)
+		(stroke
+			(width 0)
+			(type default)
+		)
+	)
 	(wire
 		(pts
@@
 				(hide yes)
 			)
+		)
+	)
+	(global_label "DISPLAY_CS"
+		(shape output)
+		(at 91.44 83.82 180)
+		(fields_autoplaced yes)
+		(effects
+			(font
+				(size 1.27 1.27)
+			)
+			(justify right)
+		)
+		(property "Intersheetrefs" "${INTERSHEET_REFS}"
+			(at 77.4481 83.82 0)
+			(effects
+				(font
+					(size 1.27 1.27)
+				)
+				(justify right)
+				(hide yes)
+			)

Commit message: 250827-1625
Connections:
- net DISPLAY_CS: no longer names the net of U1.10 (GPIO32)
Changed lines of the file:
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@@
-	(wire
-		(pts
-			(xy 91.44 83.82) (xy 113.03 83.82)
-		)
-		(stroke
-			(width 0)
-			(type default)
-		)
-	)
 	(wire
 		(pts
@@
 				(hide yes)
 			)
-		)
-	)
-	(global_label "DISPLAY_CS"
-		(shape output)
-		(at 91.44 83.82 180)
-		(fields_autoplaced yes)
-		(effects
-			(font
-				(size 1.27 1.27)
-			)
-			(justify right)
-		)
-		(property "Intersheetrefs" "${INTERSHEET_REFS}"
-			(at 77.4481 83.82 0)
-			(effects
-				(font
-					(size 1.27 1.27)
-				)
-				(justify right)
-				(hide yes)
-			)
