File: hardware/vers0.9/perifericos.kicad_sch (KiCad schematic)
At the start: 7 parts, among them J4 Conn_02x13_Odd_Even, U7 74HC244, U8 74HC374

Commit message: 250330-0836
Parts:
- removed R4: 100K, symbol Device:R
- removed U7: 74HC244, symbol 74xx:74HC244
- removed U8: 74HC374, symbol 74xx:74HC374
- added U2: 74HC00, symbol 74xx:74HC00
- added U3: TXB0108PW, Package_SO:TSSOP-20_4.4x6.5mm_P0.65mm, symbol Logic_LevelTranslator:TXB0108PW
- added U4: ~, symbol dev_boards:HC-SR08
Connections:
- net 3,3V: now also U3.2 (V_{CCA})
- net 5V: now also U3.19 (V_{CCB}); no longer R1.1
- net GND: now also J4.15 (Pin_15), U3.10 (OE), U3.11 (GND)
- net at R1.2: no longer J4.15 (Pin_15)
- net D0: no longer names the net of J4.7 (Pin_7)
- net D1: no longer names the net of J4.8 (Pin_8)
- net D2: no longer names the net of J4.9 (Pin_9)
- net D3: no longer names the net of J4.10 (Pin_10)
- net D4: no longer names the net of J4.11 (Pin_11)
- net D5: no longer names the net of J4.12 (Pin_12)
- net D6: no longer names the net of J4.13 (Pin_13)
- net D7: no longer names the net of J4.14 (Pin_14)
- net DISP_RS: no longer names the net of J4.4 (Pin_4)
- net DISP_RS: now also U3.14 (B6)
- net DISP_R/W: no longer names the net of J4.5 (Pin_5)
- net DISP_R/W: now also U3.13 (B7)
- net /DISPLAY_E: no longer names the net of J4.6 (Pin_6)
- net /DISPLAY_E: now also U3.15 (B5)
- net /RESET: no longer names the net of J4.17 (Pin_17)
- net /RESET: now also U3.12 (B8)
- new net: U2.3, U3.9 (A8)
- new net DISPLAY_CS: U3.7 (A6)
- new net DISPLAY_SCLK: U3.6 (A5)
- new net DISPLAY_SID: U3.8 (A7)
- new net RESET: U2.1, U2.2
Other:
- moved on the sheet: J4, R1

Commit message: 250404-0705
Parts:
- removed R1: 10K, symbol Device:R
- removed U2: 74HC00, symbol 74xx:74HC00
- removed U4: ~, symbol dev_boards:HC-SR08
- added C10, C11, C2, C9: 100nF, symbol Device:C
- added C5, C6, C7, C8: 10nF, symbol Device:C
- added D1, D2, D3, D4: 1N4148, Diode_THT:D_DO-35_SOD27_P7.62mm_Horizontal, symbol Diode:1N4148
- added J5: Teclado, symbol Connector_Generic:Conn_02x05_Odd_Even
- added J6: Encoders, symbol Connector_Generic:Conn_02x05_Odd_Even
- added R10, R11, R2, R3, R4, R5, R6, R7, R8, R9: 10K, symbol Device:R
- added U10: ULN2803A, symbol Transistor_Array:ULN2803A
- added U2: 74HC595, symbol 74xx:74HC595
- added U6: 74HC165, symbol 74xx:74HC165
Connections:
- net 3,3V: now also C2.1, R6.1, R7.1, U2.16 (VCC), U6.16 (VCC)
- net 5V: now also J4.4 (Pin_4), C9.1
- net GND: now also U3.1 (A1), C10.1, C11.2, C2.2, C5.2, C6.2, C7.2, C8.2, C9.2, J6.10 (Pin_10), J6.2 (Pin_2), J6.4 (Pin_4), J6.7 (Pin_7), R2.2, R3.2, R4.2, R5.2, U10.9 (GND), U2.8 (GND), U6.10 (SERIAL_INPUT), U6.15 (CLOCK_INHIBIT), U6.5 (D6), U6.6 (D7), U6.8 (GND)
- net RESET: now also U2.13 (~{OE})
- net at U3.14 (B6): now also J4.6 (Pin_6); no longer J4.4 (Pin_4)
- net at U3.15 (B5): now also U10.4 (I4); no longer J4.6 (Pin_6)
- net at U3.16 (B4): now also U10.3 (I3)
- net at U3.17 (B3): now also U10.2 (I2)
- net at U3.18 (B2): now also U10.1 (I1)
- net R1: now reaches U3.3 (A2)
- net R1: now also U2.4 (QE)
- net R2: now reaches U3.4 (A3)
- net R2: now also U2.5 (QF)
- net R3: now reaches U3.5 (A4)
- net R3: now also U2.6 (QG)
- net /RESET: now reaches U3.9 (A8)
- net /RESET: now also U2.10 (~{SRCLR})
- net DISPLAY_CS renamed DISPLAY_CLK
- net DISPLAY_SCLK renamed R4
- net R4: now also U2.7 (QH)
- net DISPLAY_SID renamed DISPLAY_DATA
- new net: J5.5 (Pin_5), R2.1, U6.11 (D0)
- new net: J5.7 (Pin_7), R3.1, U6.12 (D1)
- new net: J5.8 (Pin_8), R4.1, U6.13 (D2)
- new net: J5.6 (Pin_6), R5.1, U6.14 (D3)
- new net: C11.1, J6.1 (Pin_1), R6.2, U6.3 (D4)
- new net: C10.2, J6.9 (Pin_9), R7.2, U6.4 (D5)
- new net: D1.1 (K), J5.4 (Pin_4)
- new net: D1.2 (A), U2.15 (QA)
- new net: D3.1 (K), J5.1 (Pin_1)
- new net: D3.2 (A), U2.2 (QC)
- new net: D2.2 (A), U2.1 (QB)
- new net: D4.2 (A), U2.3 (QD)
- new net: D4.1 (K), J5.3 (Pin_3)
- new net: D2.1 (K), J5.2 (Pin_2)
- new net 12V: U10.10 (COM)
- new net E0_A: J6.3 (Pin_3), R8.2
- new net E0_B: J6.5 (Pin_5), R9.2
- new net E1_A: J6.6 (Pin_6), R10.2
- new net E1_B: J6.8 (Pin_8), R11.2
- new net ENC0_A: C7.1, R8.1
- new net ENC0_B: C8.1, R9.1
- new net ENC1_A: C5.1, R10.1
- new net ENC1_B: C6.1, R11.1
- new net RELE1: U10.18 (O1)
- new net RELE2: U10.17 (O2)
- new net RELE3: U10.16 (O3)
- new net RELE4: U10.15 (O4)
- new net SHREG_CLK: U2.11 (SRCLK), U6.2 (CLOCK)
- new net SHREG_DATAIN: U6.9 (QH)
- new net SHREG_DATAOUT: U2.14 (SER)
- new net SHREG_HOLD: U2.12 (RCLK), U6.1 (SHIFT/LOAD)
Other:
- moved on the sheet: C3, C4, U3

Commit message: 250425-1655
Connections:
- net RST: now reaches J4.17 (Pin_17), U3.12 (B8)
- net R/W: now reaches J4.5 (Pin_5), U3.13 (B7)
- net E: now reaches J4.6 (Pin_6), U3.14 (B6)
Changed lines of the file:
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@@
+		)
+	)
+	(label "PSB"
+		(at 86.36 176.53 0)
+		(effects
+			(font
+				(size 1.27 1.27)
+			)
+			(justify left bottom)
+		)
+	)
+	(label "BLK"
+		(at 106.68 181.61 0)
+		(effects
+			(font
+				(size 1.27 1.27)
+			)
+			(justify left bottom)
 		)
 	)
@@
 		)
 	)
+	(label "E"
+		(at 106.68 163.83 0)
+		(effects
+			(font
+				(size 1.27 1.27)
+			)
+			(justify left bottom)
+		)
+	)
 	(label "R2"
 		(at 40.64 118.11 0)
@@
 		)
 	)
+	(label "RS"
+		(at 106.68 161.29 0)
+		(effects
+			(font
+				(size 1.27 1.27)
+			)
+			(justify left bottom)
+		)
+	)
 	(label "R1"
 		(at 40.64 115.57 0)
@@
 		)
 	)
+	(label "R{slash}W"
+		(at 86.36 163.83 0)
+		(effects
+			(font
+				(size 1.27 1.27)
+			)
+			(justify left bottom)
+		)
+	)
 	(label "R3"
 		(at 182.88 53.34 0)
@@
 		)
 	)
+	(label "BLA"
+		(at 86.36 181.61 0)
+		(effects
+			(font
+				(size 1.27 1.27)
+			)
+			(justify left bottom)
+		)
+	)
 	(label "R4"
 		(at 40.64 123.19 0)
@@
 	(label "E1_B"
 		(at 264.16 146.05 0)
+		(effects
+			(font
+				(size 1.27 1.27)
+			)
+			(justify left bottom)
+		)
+	)
+	(label "RST"
+		(at 86.36 179.07 0)
 		(effects
 			(font
@@
 		(on_board yes)
 		(dnp no)
-		(fields_autoplaced yes)
 		(property "Reference" "#PWR13"
 			(at 78.74 163.83 0)
@@
 		)
 		(property "Value" "GND"
-			(at 78.74 162.56 0)
-			(effects
-				(font
+			(at 81.28 160.274 0)
+			(effects
+				(font

Commit message: 250427-1145
Parts:
- removed C2, C3, C4, C9: 100nF, symbol Device:C
- removed U3: TXB0108PW, Package_SO:TSSOP-20_4.4x6.5mm_P0.65mm, symbol Logic_LevelTranslator:TXB0108PW
- added U3: ~, symbol dev_boards:TXB0108_BOARD
Connections:
- net 3,3V: now also U3.1 (VCCA)
- net 5V: now also U3.20 (VCCB)
- net DISPLAY_CLK: now also U3.7 (A6)
- net DISPLAY_DATA: now also U3.8 (A7)
- net E: now also U3.14 (B6)
- net GND: now also U3.10 (OE), U3.11 (GND), U3.2 (A1)
- net R1: now also U3.3 (A2)
- net R2: now also U3.4 (A3)
- net R3: now also U3.5 (A4)
- net R4: now also U3.6 (A5)
- net RST: now also U3.12 (B8)
- net R/W: now also U3.13 (B7)
- net /RESET: now also U3.9 (A8)
- net at U10.4 (I4): now also U3.15 (B5)
- net at U10.3 (I3): now also U3.16 (B4)
- net at U10.2 (I2): now also U3.17 (B3)
- net at U10.1 (I1): now also U3.18 (B2)

Commit message: 250507-1622
Connections:
- net 3,3V: now also U3.10 (OE), U3.2 (A1)
- net GND: no longer U3.10 (OE), U3.2 (A1)
Changed lines of the file:
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@@
 	)
 	(junction
+		(at 40.64 110.49)
+		(diameter 0)
+		(color 0 0 0 0)
+	)
+	(junction
 		(at 218.44 73.66)
 		(diameter 0)
@@
 	)
 	(junction
-		(at 40.64 110.49)
-		(diameter 0)
-		(color 0 0 0 0)
-	)
-	(junction
 		(at 63.5 38.1)
 		(diameter 0)
@@
 	(wire
 		(pts
-			(xy 40.64 93.98) (xy 45.72 93.98)
-		)
-		(stroke
-			(width 0)
-			(type default)
-		)
-	)
-	(wire
-		(pts
 			(xy 132.08 88.9) (xy 132.08 157.48)
 		)
@@
 		)
 	)
-	(wire
-		(pts
-			(xy 45.72 93.98) (xy 45.72 97.79)
-		)
-		(stroke
-			(width 0)
-			(type default)
-		)
-	)
 	(bus
 		(pts
@@
 	(wire
 		(pts
+			(xy 40.64 99.06) (xy 40.64 110.49)
+		)
+		(stroke
+			(width 0)
+			(type default)
+		)
+	)
+	(wire
+		(pts
 			(xy 66.04 123.19) (xy 91.44 123.19)
 		)
@@
 	(wire
 		(pts
-			(xy 40.64 93.98) (xy 40.64 110.49)
-		)
-		(stroke
-			(width 0)
-			(type default)
-		)
-	)
-	(wire
-		(pts
 			(xy 222.25 148.59) (xy 224.79 148.59)
 		)
@@
 		)
 	)
-	(label "RS"
+	(label "CS"
 		(at 106.68 161.29 0)
 		(effects
@@
 	(symbol
 		(lib_id "power:GND")
-		(at 45.72 97.79 0)
-		(unit 1)
-		(exclude_from_sim no)
-		(in_bom yes)
-		(on_board yes)
-		(dnp no)
-		(fields_autoplaced yes)
-		(property "Reference" "#PWR17"
-			(at 45.72 104.14 0)
-			(effects
-				(font
-					(size 1.27 1.27)
-				)
-				(hide yes)
-			)
-		)
-		(property "Value" "GND"
-			(at 45.72 102.87 0)
-			(effects
-				(font
-					(size 1.27 1.27)
-				)
-			)
-		)
-		(property "Footprint" ""
-			(at 45.72 97.79 0)
-			(effects
-				(font
-					(size 1.27 1.27)
-				)
-				(hide yes)
-			)
-		)
-		(property "Datasheet" ""
-			(at 45.72 97.79 0)
-			(effects
-				(font
-					(size 1.27 1.27)
-				)
-				(hide yes)
-			)
-		)
-		(property "Description" "Power symbol creates a global label with name \"GND\" , ground"
-			(at 45.72 97.79 0)
-			(effects
-				(font
-					(size 1.27 1.27)
-				)
-				(hide yes)
-			)
-		)
-		(pin "1"
-		)
-		(instances
-			(project "gerador_sinais"
-				(path "/1aec9b5d-f0c7-4911-a832-6f11be903841/5ad42e96-ca87-4402-a9ee-0c3f738ace78"
-					(reference "#PWR17")
-					(unit 1)
-				)
-			)
-		)
-	)
-	(symbol
-		(lib_id "power:GND")
 		(at 265.43 149.86 0)
 		(unit 1)
@@
 					(unit 1)
 				)
+			)
+		)
+	)
+	(symbol
+		(lib_id "power:VCC")
+		(at 40.64 99.06 0)
+		(unit 1)
+		(exclude_from_sim no)
+		(in_bom yes)
+		(on_board yes)
+		(dnp no)
+		(fields_autoplaced yes)
+		(property "Reference" "#PWR17"
+			(at 40.64 102.87 0)
+			(effects
+				(font
+					(size 1.27 1.27)
+				)
+				(hide yes)
+			)
+		)
+		(property "Value" "3,3V"
+			(at 40.64 93.98 0)
+			(effects
+				(font
+					(size 1.27 1.27)
+				)
+			)
+		)
+		(property "Footprint" ""
+			(at 40.64 99.06 0)
+			(effects
+				(font
+					(size 1.27 1.27)
+				)
+				(hide yes)
+			)
+		)
+		(property "Datasheet" ""
+			(at 40.64 99.06 0)
+			(effects
+				(font
+					(size 1.27 1.27)
+				)
+				(hide yes)
+			)
+		)
+		(property "Description" "Power symbol creates a global label with name \"VCC\""
+			(at 40.64 99.06 0)
+			(effects
+				(font
+					(size 1.27 1.27)
+				)
+				(hide yes)
+			)
+		)
+		(pin "1"
+		)
+		(instances
+			(project "gerador_sinais"
+				(path "/1aec9b5d-f0c7-4911-a832-6f11be903841/5ad42e96-ca87-4402-a9ee-0c3f738ace78"
+					(reference "#PWR17")
+					(unit 1)
+				)

Commit message: 250826-1410
Parts:
- added RV1: 4K, symbol Device:R_Potentiometer_Trim_US
Connections:
- net 3,3V: no longer U3.2 (A1)
- net 5V: no longer J4.4 (Pin_4)
- net GND: now also RV1.3
- net VOUT: now reaches J4.18 (Pin_18)
- net VOUT: now also RV1.1
- net at J4.3 (Pin_3): now also RV1.2
- net CS: now reaches U3.19 (B1)
- net CS: now also J4.4 (Pin_4)
- new net DISPLAY_CS: U3.2 (A1)
Other:
- moved on the sheet: U10, U3

Commit message: 250827-1625
Parts:
- removed U3: ~, symbol dev_boards:TXB0108_BOARD
- added U11: ~, symbol dev_boards:TXB0108_BOARD
Connections:
- net CS is gone; now on net 3,3V: J4.4 (Pin_4)
- net E is gone; now on net DISPLAY_CLK: J4.6 (Pin_6)
- net RST is gone; now on net /RESET: J4.17 (Pin_17)
- net R/W is gone; now on net DISPLAY_DATA: J4.5 (Pin_5)
- net 3,3V: now also J4.19 (Pin_19), J4.2 (Pin_2), U11.1 (VCCA), U11.10 (OE)
- net 5V: now also RV1.1, U11.20 (VCCB); no longer J4.19 (Pin_19), J4.2 (Pin_2)
- net GND: now also U11.11 (GND)
- net R1: now also U11.2 (A1)
- net R2: now also U11.3 (A2)
- net R3: now also U11.4 (A3)
- net R4: now also U11.5 (A4)
- net at U10.4 (I4): now also U11.16 (B4)
- net at U10.3 (I3): now also U11.17 (B3)
- net at U10.2 (I2): now also U11.18 (B2)
- net at U10.1 (I1): now also U11.19 (B1)
- net VOUT: no longer names the net of J4.18 (Pin_18)
- net VOUT: no longer RV1.1
Other:
- moved on the sheet: J4, RV1

Commit message: 250829-1845
Parts:
- R2, R3, R4, R5: value 10K -> 22K
Connections:
- net 3,3V: now also U6.10 (SERIAL_INPUT)
- net GND: no longer U6.10 (SERIAL_INPUT)
- net at R2.1, U6.11 (D0): now also J5.7 (Pin_7); no longer J5.5 (Pin_5)
- net at R3.1, U6.12 (D1): now also J5.9 (Pin_9); no longer J5.7 (Pin_7)
- net at D3.1 (K): now also J5.3 (Pin_3); no longer J5.1 (Pin_1)
- net at D4.1 (K): now also J5.5 (Pin_5); no longer J5.3 (Pin_3)
Other:
- note added: "*R8 do display foi desconectado"
- moved on the sheet: R2, R3
